File: PCB/MIDIWidgetRevD.brd (EAGLE design)
At the start: 43.2 x 83.8 mm, 69 parts, among them CN1 10118192-0001LF, U1 SN74ACT373PWR, U2 SN74ACT373PWR, U3 SN74ACT373PWR, U4 ATMEGA32U2-AU, U5 PC900V0NIPXF, U6 SN74LVC1G17DBVR, U7 TPS2113APWR, U8 LM2734Y, Y1 403C35E16M00000

Commit message: PCB Rev D
Connections:
- net VIN-RECT renamed VIN
Routing:
- net USBVCC: track 3.93 -> 10.7 mm
- net D2/PDI: track 63.5 -> 69.3 mm
- net D5: track 60.9 -> 65.0 mm
- net VREG: track 45.5 -> 49.1 mm
- net D6: track 60.5 -> 63.8 mm
- net D3/PDO: track 72.0 -> 75.0 mm
- net D4: track 74.4 -> 77.4 mm
- net MIDI-TX: track 36.8 -> 39.0 mm
- net D1/SCK: track 65.4 -> 67.4 mm
- net D7: track 58.6 -> 60.5 mm
- net +5V: track 232.1 -> 234.0 mm
- net MIDI-RX: track 47.0 -> 48.5 mm
- net D0: track 62.5 -> 63.7 mm
Other:
- board text added: "MIDIWIDGET REV D"
- board text added: "MIDIWidget copyright 2015-2017 John Staskevich john@codeandcopper.com This work is licensed under a Creative Commons Attribution 4.0 International License. http://creativecommons.org/licenses/by/4.0/"
- board text removed: "MIDIWIDGET REV B"
- board text removed: "MIDIWIDGET.COM"
