File: PCB/MIDIWidgetRevD.sch (EAGLE design)
At the start: 69 parts, among them CN1 10118192-0001LF, U1 SN74ACT373PWR, U2 SN74ACT373PWR, U3 SN74ACT373PWR, U4 ATMEGA32U2-AU, U5 PC900V0NIPXF, U6 SN74LVC1G17DBVR, U7 TPS2113APWR, U8 LM2734Y, Y1 403C35E16M00000

Commit message: PCB Rev D
Connections:
- net VIN-RECT renamed VIN
Other:
- note added: "MIDIWidget copyright 2015-2017 John Staskevich john@codeandcopper.com This work is licensed under a Creative Commons Attribution 4.0 International License. http://creativecommons.org/licenses/by/4.0/"
- note removed: "5V REGULATOR"
- note removed: "ACT/STBY LEDS"
- note removed: "CRYSTAL"
- note removed: "ICSP CONTACTS"
- note removed: "MICROCONTROLLER"
- note removed: "MIDI PORTS"
- note removed: "MIDIWidget www.midiwidget.com copyright John Staskevich, 2015 john@codeandcopper.com This work is licensed under a Creative Commons Attribution 4.0 International License. http://creativecommons.org/licenses/by/4.0/"
- note removed: "OUTPUT LATCHES"
- note removed: "POWER MUX"
- note removed: "POWER/SWITCH HEADER"
- note removed: "USB PORT"
- moved on the sheet: C1, C11, C12, C13, C14, C15, C16, C17, C18, C19, C2, C20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
